File: SoilProbe/SoilProbe.sch (KiCad schematic (older format))
At the start: 3 parts

Commit message: Tests
Tests
Parts:
- P1: renamed from P?; footprint (none) -> Connectors:bornier2
- gave numbers to parts that had none: 2
Changed lines of the file:
@@
 LIBS:contrib
 LIBS:valves
+LIBS:SoilProbe-cache
 EELAYER 25 0
 EELAYER END
@@
 $EndDescr
 $Comp
-L CONN_01X02 P?
+L CONN_01X02 P1
 U 1 1 58D97786
 P 2700 2700
-F 0 "P?" H 2700 2850 50  0000 C CNN
+F 0 "P1" H 2700 2850 50  0000 C CNN
 F 1 "CONN_01X02" V 2800 2700 50  0000 C CNN
-F 2 "" H 2700 2700 50  0000 C CNN
+F 2 "Connectors:bornier2" H 2700 2700 50  0000 C CNN
 F 3 "" H 2700 2700 50  0000 C CNN
 	1    2700 2700
@@
 $EndComp
 $Comp
-L CONN_01X01 P?
+L CONN_01X01 P2
 U 1 1 58D977BC
 P 3350 3500
-F 0 "P?" H 3350 3600 50  0000 C CNN
+F 0 "P2" H 3350 3600 50  0000 C CNN
 F 1 "CONN_01X01" V 3450 3500 50  0000 C CNN
 F 2 "" H 3350 3500 50  0000 C CNN
@@
 $EndComp
 $Comp
-L CONN_01X01 P?
+L CONN_01X01 P3
 U 1 1 58D977FF
 P 4050 3500
-F 0 "P?" H 4050 3600 50  0000 C CNN
+F 0 "P3" H 4050 3600 50  0000 C CNN
 F 1 "CONN_01X01" V 4150 3500 50  0000 C CNN
 F 2 "" H 4050 3500 50  0000 C CNN
